File: LiPoBCB-V2.kicad_sch (KiCad schematic)
At the start: 27 parts, among them J1 USB-C_6_pin_receptacle, J2 Conn_01x02, Q1 Q_Dual_PMOS_S1G1D2S2G2D1, U1 ETA9740

Commit message: Adds new solder connector footprints
Parts:
- P1: renamed from TP1; value 5V -> Solder Pad; footprint TestPoint:TestPoint_THTPad_2.5x2.5mm_Drill1.2mm -> LiPoBCB-V2:TestPoint_THTPad_2.5x2.5mm_Drill1.2mm; symbol Connector:TestPoint -> LiPoBCB-V2:Solder Pad
- P2: renamed from TP2; value GND -> Solder Pad; footprint TestPoint:TestPoint_THTPad_2.5x2.5mm_Drill1.2mm -> LiPoBCB-V2:TestPoint_THTPad_2.5x2.5mm_Drill1.2mm; symbol Connector:TestPoint -> LiPoBCB-V2:Solder Pad
Changed lines of the file:
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@@
     (pin "5")
   )
-  (symbol (lib_id "Connector:TestPoint") (at 101.6 57.15 90) (unit 1)
-    (in_bom yes) (on_board yes)
-    (property "Reference" "TP2" (id 0) (at 90.17 57.15 90))
-    (property "Value" "GND" (id 1) (at 93.98 57.15 90))
-    (property "Footprint" "TestPoint:TestPoint_THTPad_2.5x2.5mm_Drill1.2mm" (id 2) (at 101.6 52.07 0)
+  (symbol (lib_id "LiPoBCB-V2:Solder Pad") (at 101.6 57.15 90) (unit 1)
+    (in_bom yes) (on_board yes)
+    (property "Reference" "P2" (id 0) (at 95.25 57.15 90))
+    (property "Value" "Solder Pad" (id 1) (at 97.79 60.96 90)
+      (effects (font (size 1.27 1.27)) hide)
+    )
+    (property "Footprint" "LiPoBCB-V2:TestPoint_THTPad_2.5x2.5mm_Drill1.2mm" (id 2) (at 101.6 52.07 0)
       (effects (font (size 1.27 1.27)) hide)
     )
@@
     (pin "2")
   )
-  (symbol (lib_id "Connector:TestPoint") (at 101.6 54.61 90) (unit 1)
-    (in_bom yes) (on_board yes)
-    (property "Reference" "TP1" (id 0) (at 90.17 54.61 90))
-    (property "Value" "5V" (id 1) (at 93.98 54.61 90))
-    (property "Footprint" "TestPoint:TestPoint_THTPad_2.5x2.5mm_Drill1.2mm" (id 2) (at 101.6 49.53 0)
+  (symbol (lib_id "LiPoBCB-V2:Solder Pad") (at 101.6 54.61 90) (unit 1)
+    (in_bom yes) (on_board yes)
+    (property "Reference" "P1" (id 0) (at 95.25 54.61 90))
+    (property "Value" "Solder Pad" (id 1) (at 97.79 50.8 90))
+    (property "Footprint" "LiPoBCB-V2:TestPoint_THTPad_2.5x2.5mm_Drill1.2mm" (id 2) (at 101.6 49.53 0)
       (effects (font (size 1.27 1.27)) hide)
     )
@@
       (reference "L1") (unit 1) (value "1 uH") (footprint "LiPoBCB-V2:L_smd_1616")
     )
+    (path "/970e99f5-6d1d-48db-a6d5-9070653e7b35"
+      (reference "P1") (unit 1) (value "Solder Pad") (footprint "LiPoBCB-V2:TestPoint_THTPad_2.5x2.5mm_Drill1.2mm")
+    )
+    (path "/28c7823c-4dc0-491b-8b7a-dabb0bc8da0f"
+      (reference "P2") (unit 1) (value "Solder Pad") (footprint "LiPoBCB-V2:TestPoint_THTPad_2.5x2.5mm_Drill1.2mm")
+    )
     (path "/21e95954-03e5-4805-be0a-a9c38dfbcf7f"
       (reference "Q1") (unit 1) (value "Q_Dual_PMOS_S1G1D2S2G2D1") (footprint "Package_TO_SOT_SMD:SOT-23-6")
@@
       (reference "R7") (unit 1) (value "10K") (footprint "Resistor_SMD:R_0603_1608Metric")
     )
-    (path "/970e99f5-6d1d-48db-a6d5-9070653e7b35"
-      (reference "TP1") (unit 1) (value "5V") (footprint "TestPoint:TestPoint_THTPad_2.5x2.5mm_Drill1.2mm")
-    )
-    (path "/28c7823c-4dc0-491b-8b7a-dabb0bc8da0f"
-      (reference "TP2") (unit 1) (value "GND") (footprint "TestPoint:TestPoint_THTPad_2.5x2.5mm_Drill1.2mm")
-    )
     (path "/8c677a46-0320-4920-b6ab-a463e7a44329"

Commit message: Adds silkscreen to the back
Parts:
- removed P1, P2: Solder Pad, LiPoBCB-V2:TestPoint_THTPad_2.5x2.5mm_Drill1.2mm, symbol LiPoBCB-V2:Solder Pad
- added P1: Solder_Connector_X2, LiPoBCB-V2:Solder_Connector_X2, symbol LiPoBCB-V2:Solder_Connector_X2
- J2: footprint Connector_PinHeader_2.54mm:PinHeader_1x02_P2.54mm_Vertical -> LiPoBCB-V2:Solder_Connector_SW
Connections:
- net GND: now also P1.2 (GND)
- net VBUS: now also P1.1 (5V)
Changed lines of the file:
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@@
+    (pin "2")
+  )
+  (symbol (lib_id "LiPoBCB-V2:Solder_Connector_X2") (at 101.6 54.61 0) (unit 1)
+    (in_bom yes) (on_board yes) (fields_autoplaced)
+    (property "Reference" "P1" (id 0) (at 98.2853 48.26 0))
+    (property "Value" "Solder_Connector_X2" (id 1) (at 98.2853 50.8 0))
+    (property "Footprint" "LiPoBCB-V2:Solder_Connector_X2" (id 2) (at 101.6 60.325 0)
+      (effects (font (size 1.27 1.27)) hide)
+    )
+    (property "Datasheet" "~" (id 3) (at 106.68 54.61 0)
+      (effects (font (size 1.27 1.27)) hide)
+    )
+    (pin "1")
     (pin "2")
   )
@@
     (pin "5")
   )
-  (symbol (lib_id "LiPoBCB-V2:Solder Pad") (at 101.6 57.15 90) (unit 1)
-    (in_bom yes) (on_board yes)
-    (property "Reference" "P2" (id 0) (at 95.25 57.15 90))
-    (property "Value" "Solder Pad" (id 1) (at 97.79 60.96 90)
-      (effects (font (size 1.27 1.27)) hide)
-    )
-    (property "Footprint" "LiPoBCB-V2:TestPoint_THTPad_2.5x2.5mm_Drill1.2mm" (id 2) (at 101.6 52.07 0)
-      (effects (font (size 1.27 1.27)) hide)
-    )
-    (property "Datasheet" "~" (id 3) (at 101.6 52.07 0)
-      (effects (font (size 1.27 1.27)) hide)
-    )
-    (pin "1")
-  )
   (symbol (lib_id "Device:R") (at 186.69 114.3 0) (unit 1)
     (in_bom yes) (on_board yes) (fields_autoplaced)
@@
     (property "Reference" "J2" (id 0) (at 93.98 104.14 0))
     (property "Value" "Conn_01x02" (id 1) (at 93.98 106.68 0))
-    (property "Footprint" "Connector_PinHeader_2.54mm:PinHeader_1x02_P2.54mm_Vertical" (id 2) (at 93.98 110.49 0)
+    (property "Footprint" "LiPoBCB-V2:Solder_Connector_SW" (id 2) (at 93.98 110.49 0)
       (effects (font (size 1.27 1.27)) hide)
     )
@@
     (pin "2")
   )
-  (symbol (lib_id "LiPoBCB-V2:Solder Pad") (at 101.6 54.61 90) (unit 1)
-    (in_bom yes) (on_board yes)
-    (property "Reference" "P1" (id 0) (at 95.25 54.61 90))
-    (property "Value" "Solder Pad" (id 1) (at 97.79 50.8 90))
-    (property "Footprint" "LiPoBCB-V2:TestPoint_THTPad_2.5x2.5mm_Drill1.2mm" (id 2) (at 101.6 49.53 0)
-      (effects (font (size 1.27 1.27)) hide)
-    )
-    (property "Datasheet" "~" (id 3) (at 101.6 49.53 0)
-      (effects (font (size 1.27 1.27)) hide)
-    )
-    (pin "1")
-  )
   (symbol (lib_id "power:+5V") (at 162.56 83.82 0) (unit 1)
     (in_bom yes) (on_board yes) (fields_autoplaced)
@@
     (pin "B5")
     (pin "B9")
-    (pin "S1")
+    (pin "S")
   )
   (symbol (lib_id "Mechanical:MountingHole") (at 140.97 52.07 0) (unit 1)
@@
     )
     (path "/3ea89e3b-438c-4e25-afed-9cebb5a00e70"
-      (reference "J2") (unit 1) (value "Conn_01x02") (footprint "Connector_PinHeader_2.54mm:PinHeader_1x02_P2.54mm_Vertical")
+      (reference "J2") (unit 1) (value "Conn_01x02") (footprint "LiPoBCB-V2:Solder_Connector_SW")
     )
     (path "/728557f3-2803-49a5-abbb-fdd88a8dc19e"
       (reference "L1") (unit 1) (value "1 uH") (footprint "LiPoBCB-V2:L_smd_1616")
     )
-    (path "/970e99f5-6d1d-48db-a6d5-9070653e7b35"
-      (reference "P1") (unit 1) (value "Solder Pad") (footprint "LiPoBCB-V2:TestPoint_THTPad_2.5x2.5mm_Drill1.2mm")
-    )
-    (path "/28c7823c-4dc0-491b-8b7a-dabb0bc8da0f"
-      (reference "P2") (unit 1) (value "Solder Pad") (footprint "LiPoBCB-V2:TestPoint_THTPad_2.5x2.5mm_Drill1.2mm")
+    (path "/178def00-c160-40e5-88c3-4419efbce1d6"
+      (reference "P1") (unit 1) (value "Solder_Connector_X2") (footprint "LiPoBCB-V2:Solder_Connector_X2")
     )
     (path "/21e95954-03e5-4805-be0a-a9c38dfbcf7f"
